File: hardware/pcb/sensor/sensor.kicad_sch (KiCad schematic)
At the start: 10 parts

Commit message: sensor,tag: Update PCB wiring to avoid bootstrap pins.
Connections:
- net at CAN_Transreceiver1.3 (CAN_RX): now also ESP32_UWB1.28 (IO16); no longer ESP32_UWB1.5 (IO2)
- net at CAN_Transreceiver1.4 (CAN_TX): now also ESP32_UWB1.27 (IO5); no longer ESP32_UWB1.6 (IO12)
Other:
- moved on the sheet: CAN_Transreceiver1
Changed lines of the file:
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@@
 		(title "Autocam Sensor")
 		(date "2025-03-27")
-		(rev "v0.4")
+		(rev "v0.5")
 	)
 	(junction
-		(at 105.41 90.17)
+		(at 129.54 90.17)
 		(diameter 0)
 		(color 0 0 0 0)
@@
 	(wire
 		(pts
+			(xy 153.67 66.04) (xy 153.67 73.66)
+		)
+		(stroke
+			(width 0)
+			(type default)
+		)
+	)
+	(wire
+		(pts
+			(xy 167.64 78.74) (xy 167.64 107.95)
+		)
+		(stroke
+			(width 0)
+			(type default)
+		)
+	)
+	(wire
+		(pts
 			(xy 93.98 120.65) (xy 101.6 120.65)
 		)
@@
 	(wire
 		(pts
+			(xy 151.13 78.74) (xy 167.64 78.74)
+		)
+		(stroke
+			(width 0)
+			(type default)
+		)
+	)
+	(wire
+		(pts
 			(xy 104.14 125.73) (xy 104.14 130.81)
 		)
@@
 	(wire
 		(pts
-			(xy 107.95 92.71) (xy 137.16 92.71)
-		)
-		(stroke
-			(width 0)
-			(type default)
-		)
-	)
-	(wire
-		(pts
-			(xy 105.41 83.82) (xy 105.41 90.17)
-		)
-		(stroke
-			(width 0)
-			(type default)
-		)
-	)
-	(wire
-		(pts
-			(xy 110.49 100.33) (xy 137.16 100.33)
+			(xy 170.18 105.41) (xy 162.56 105.41)
+		)
+		(stroke
+			(width 0)
+			(type default)
+		)
+	)
+	(wire
+		(pts
+			(xy 148.59 66.04) (xy 148.59 78.74)
+		)
+		(stroke
+			(width 0)
+			(type default)
+		)
+	)
+	(wire
+		(pts
+			(xy 170.18 73.66) (xy 170.18 105.41)
+		)
+		(stroke
+			(width 0)
+			(type default)
+		)
+	)
+	(wire
+		(pts
+			(xy 133.35 78.74) (xy 133.35 92.71)
 		)
 		(stroke
@@
 	(wire
 		(pts
-			(xy 107.95 83.82) (xy 107.95 92.71)
-		)
-		(stroke
-			(width 0)
-			(type default)
-		)
-	)
-	(wire
-		(pts
 			(xy 106.68 128.27) (xy 106.68 135.89)
 		)
@@
 	(wire
 		(pts
-			(xy 105.41 90.17) (xy 137.16 90.17)
-		)
-		(stroke
-			(width 0)
-			(type default)
-		)
-	)
-	(wire
-		(pts
-			(xy 101.6 90.17) (xy 105.41 90.17)
+			(xy 146.05 66.04) (xy 146.05 74.93)
+		)
+		(stroke
+			(width 0)
+			(type default)
+		)
+	)
+	(wire
+		(pts
+			(xy 148.59 78.74) (xy 133.35 78.74)
+		)
+		(stroke
+			(width 0)
+			(type default)
+		)
+	)
+	(wire
+		(pts
+			(xy 129.54 90.17) (xy 137.16 90.17)
+		)
+		(stroke
+			(width 0)
+			(type default)
+		)
+	)
+	(wire
+		(pts
+			(xy 129.54 74.93) (xy 146.05 74.93)
+		)
+		(stroke
+			(width 0)
+			(type default)
+		)
+	)
+	(wire
+		(pts
+			(xy 101.6 90.17) (xy 129.54 90.17)
+		)
+		(stroke
+			(width 0)
+			(type default)
+		)
+	)
+	(wire
+		(pts
+			(xy 167.64 107.95) (xy 162.56 107.95)
 		)
 		(stroke
@@
 	(wire
 		(pts
+			(xy 153.67 73.66) (xy 170.18 73.66)
+		)
+		(stroke
+			(width 0)
+			(type default)
+		)
+	)
+	(wire
+		(pts
 			(xy 125.73 128.27) (xy 137.16 128.27)
 		)
@@
 	(wire
 		(pts
+			(xy 151.13 66.04) (xy 151.13 78.74)
+		)
+		(stroke
+			(width 0)
+			(type default)
+		)
+	)
+	(wire
+		(pts
 			(xy 125.73 125.73) (xy 137.16 125.73)
 		)
@@
 	(wire
 		(pts
-			(xy 110.49 83.82) (xy 110.49 100.33)
-		)
-		(stroke
-			(width 0)
-			(type default)
-		)
-	)
-	(wire
-		(pts
-			(xy 113.03 102.87) (xy 137.16 102.87)
-		)
-		(stroke
-			(width 0)
-			(type default)
-		)
-	)
-	(wire
-		(pts
 			(xy 118.11 128.27) (xy 106.68 128.27)
 		)
@@
 	(wire
 		(pts
-			(xy 113.03 83.82) (xy 113.03 102.87)
-		)
-		(stroke
-			(width 0)
-			(type default)
-		)
-	)
-	(wire
-		(pts
 			(xy 213.36 101.6) (xy 213.36 92.71)
+		)
+		(stroke
+			(width 0)
+			(type default)
+		)
+	)
+	(wire
+		(pts
+			(xy 133.35 92.71) (xy 137.16 92.71)
+		)
+		(stroke
+			(width 0)
+			(type default)
+		)
+	)
+	(wire
+		(pts
+			(xy 129.54 74.93) (xy 129.54 90.17)
 		)
 		(stroke
@@
 	(symbol
 		(lib_id "autocam:Waveshare_CAN_transreceiver")
-		(at 105.41 78.74 90)
+		(at 146.05 60.96 90)
 		(unit 1)
 		(exclude_from_sim no)
@@
 		(dnp no)
 		(property "Reference" "CAN_Transreceiver1"
-			(at 99.06 66.4367 0)
+			(at 139.7 48.6567 0)
 			(effects
 				(font
@@
 		)
 		(property "Value" "~"
-			(at 101.6 66.4367 0)
+			(at 142.24 48.6567 0)
 			(effects
 				(font
@@
 		)
 		(property "Footprint" "Autocam:Waveshare CAN Transreceiver"
-			(at 105.41 78.74 0)
+			(at 146.05 60.96 0)
 			(effects
 				(font
@@
 		)
 		(property "Datasheet" ""
-			(at 105.41 78.74 0)
+			(at 146.05 60.96 0)
 			(effects
 				(font
@@
 		)
 		(property "Description" ""
-			(at 105.41 78.74 0)
-			(effects
-				(font
+			(at 146.05 60.96 0)
+			(effects
+				(font
