File: hardware/pcb/server/server.kicad_pcb (KiCad board)
At the start: 2 copper layers, 52.1 x 57.2 mm, 15 parts

Commit message: hardware/pcb/server: Update pcb pins for the server.
Update the wiring accordingly to use D2-D8 pins.
Parts:
- moved ESP32_Nano1 38.7 mm to (146.1, 115.6), turned to 90 degrees
- moved R1 2.54 mm to (149.0, 95.2)
- moved R3 2.54 mm to (149.0, 100.3)
- moved R5 2.54 mm to (149.0, 105.4)
- moved R2 2.54 mm to (149.0, 97.8)
- moved R4 2.54 mm to (149.0, 102.9)
Connections:
- ESP32_Nano1 pad 10: unconnected-(ESP32_Nano1-D7-Pad10) -> Net-(2_PIN_CONNECTOR2-Pin_2)
- ESP32_Nano1 pad 11: unconnected-(ESP32_Nano1-D8-Pad11) -> Net-(2_PIN_CONNECTOR2-Pin_1)
- ESP32_Nano1 pad 19: Net-(ESP32_Nano1-A0) -> unconnected-(ESP32_Nano1-A0-Pad19)
- ESP32_Nano1 pad 20: Net-(ESP32_Nano1-A1) -> unconnected-(ESP32_Nano1-A1-Pad20)
- ESP32_Nano1 pad 21: Net-(ESP32_Nano1-A2) -> unconnected-(ESP32_Nano1-A2-Pad21)
- ESP32_Nano1 pad 22: Net-(ESP32_Nano1-A3) -> unconnected-(ESP32_Nano1-A3-Pad22)
- ESP32_Nano1 pad 23: Net-(ESP32_Nano1-A4) -> unconnected-(ESP32_Nano1-A4-Pad23)
- ESP32_Nano1 pad 24: Net-(2_PIN_CONNECTOR2-Pin_2) -> unconnected-(ESP32_Nano1-A5-Pad24)
- ESP32_Nano1 pad 25: Net-(2_PIN_CONNECTOR2-Pin_1) -> unconnected-(ESP32_Nano1-A6-Pad25)
- ESP32_Nano1 pad 5: unconnected-(ESP32_Nano1-D2-Pad5) -> Net-(ESP32_Nano1-D2)
- ESP32_Nano1 pad 6: unconnected-(ESP32_Nano1-D3-Pad6) -> Net-(ESP32_Nano1-D3)
- ESP32_Nano1 pad 7: unconnected-(ESP32_Nano1-D4-Pad7) -> Net-(ESP32_Nano1-D4)
- ESP32_Nano1 pad 8: unconnected-(ESP32_Nano1-D5-Pad8) -> Net-(ESP32_Nano1-D5)
- ESP32_Nano1 pad 9: unconnected-(ESP32_Nano1-D6-Pad9) -> Net-(ESP32_Nano1-D6)
- R1 pad 1: Net-(ESP32_Nano1-A4) -> Net-(ESP32_Nano1-D6)
- R2 pad 1: Net-(ESP32_Nano1-A3) -> Net-(ESP32_Nano1-D5)
- R3 pad 1: Net-(ESP32_Nano1-A2) -> Net-(ESP32_Nano1-D4)
- R4 pad 1: Net-(ESP32_Nano1-A1) -> Net-(ESP32_Nano1-D3)
- R5 pad 1: Net-(ESP32_Nano1-A0) -> Net-(ESP32_Nano1-D2)
Routing:
- net Net-(2_PIN_CONNECTOR1-Pin_1): track 5.12 -> 64.5 mm
- net Net-(2_PIN_CONNECTOR1-Pin_2): track 11.3 -> 66.9 mm
- net Net-(ESP32_Nano1-3.3V): track 54.4 -> 64.8 mm
- net Net-(ESP32_Nano1-D6): track 0.00 -> 2.94 mm
- net Net-(ESP32_Nano1-D5): track 0.00 -> 2.94 mm
- net Net-(ESP32_Nano1-D4): track 0.00 -> 2.94 mm
- net Net-(ESP32_Nano1-D3): track 0.00 -> 2.94 mm
- net Net-(ESP32_Nano1-D2): track 0.00 -> 2.94 mm
- net Net-(ESP32_Nano1-A4): track 2.94 -> 0.00 mm
- net Net-(ESP32_Nano1-A3): track 2.94 -> 0.00 mm
- net Net-(ESP32_Nano1-A2): track 2.94 -> 0.00 mm
- net Net-(ESP32_Nano1-A1): track 2.94 -> 0.00 mm
- net Net-(ESP32_Nano1-A0): track 2.94 -> 0.00 mm
- net Net-(RGB_LED_ROUND1-R): track 13.7 -> 10.8 mm
- net Net-(RGB_LED_ROUND3-B): track 10.1 -> 12.6 mm
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Other:
- board text added: "v0.3"
- board text removed: "v0.2"
